Commit message: Add UR + Robotiq 2F-85 gz bringup + self-describing gripper config
- ur_gripper_gz: UR + PickNik 2F-85 (vendor robotiq_description geometry) gz_ros2_control
  bringup (urdf/config/launch). REQUIRES the bullet-featherstone physics engine: gz Harmonic's
  default DART engine has no mimic-constraint support, which was the root cause of the gripper
  mimic failures (Hand-E and 2F-85). The launch forces it. The gripper is a GripperActionController
  (gripper_cmd), matching ur_control gripper_type='85'. Verified: arm move + gripper close + all
  5 mimic joints articulate.
- ur_control/gripper_configs.py: gripper registry (robotiq_2f85, robotiq_hande) +
  apply_gripper_config() + read_active_gripper() (latched /active_gripper topic).
- ur_control_examples: --gripper accepts a registry name or 'auto' (reads /active_gripper
  published by the bringup) -> resolves the client config internally, no --params-file needed.
- grippers.py: actionable error when gripper params are missing.
- Hand-E: cap finger travel to a jam-free range [0.002, 0.02] + spawn inside it; client config.

Co-Authored-By: Claude Opus 4.8 (1M context) <noreply@anthropic.com>

File: ur_gripper_gz/urdf/inc/robotiq_hande_gripper.xacro (robot description, xacro)
@@ -79,4 +79,8 @@
       </collision>
     </link>
+    <!-- Travel capped to a jam-free range for gz: the real Hand-E stroke is 0..0.025 per
+         finger, but in gz the fingers interpenetrate (jam) near the fully-open (0) and
+         fully-closed (>~0.022) extremes. gz physics enforces these joint limits, so even
+         raw FollowJointTrajectory goals beyond them are clamped. -->
     <joint name="${prefix}finger_joint" type="prismatic">
       <origin rpy="0 0 0" xyz="0 0 0.099"/>
@@ -84,5 +88,5 @@
       <child link="${prefix}hande_left_finger"/>
       <axis xyz="-1 0 0"/>
-      <limit effort="130" lower="0" upper="0.025" velocity="0.15"/>
+      <limit effort="130" lower="0.002" upper="0.02" velocity="0.15"/>
     </joint>
     <!-- NOTE (gz): the real Hand-E has one actuator + a mimic finger, but gz Harmonic's
@@ -95,5 +99,5 @@
       <child link="${prefix}hande_right_finger"/>
       <axis xyz="1 0 0"/>
-      <limit effort="130" lower="0" upper="0.025" velocity="0.15"/>
+      <limit effort="130" lower="0.002" upper="0.02" velocity="0.15"/>
     </joint>
   </xacro:macro>

File: ur_gripper_gz/urdf/ur_gripper_hande_gz.urdf.xacro (robot description, xacro)
@@ -67,4 +67,4 @@
       wrist_2_joint=-1.57,
       wrist_3_joint=0.0)}"
-    finger_initial_position="0.0"/>
+    finger_initial_position="0.002"/>
 </robot>

Commit message: Restore Hand-E single-actuator + mimic (bullet-featherstone); publish-once /active_gripper
Now that the mimic root cause is known (gz Harmonic needs bullet-featherstone), revert the
Hand-E from the independent-dual-command workaround to the real single-actuator design:
- robotiq_hande_gripper.xacro: hande_right_finger_joint mimics finger_joint again.
- ur_gripper_hande.ros2_control.xacro: mimic finger is state-only (no command interface).
- ur_gz_controllers.yaml: gripper_controller drives only finger_joint.
- grippers.py: Hand-E trajectory commands only finger_joint.
- ur_gz_control.launch.py: force the bullet-featherstone physics engine.
Verified in gz: both fingers articulate via the mimic (close L=R~0.019, open L=R~0.002).

Also replace the 1 Hz  /active_gripper latch (which spammed 'publishing #N')
with a small active_gripper_publisher node that publishes ONCE (transient-local) and stays
alive; used by both the Hand-E and 2F-85 launches.

Co-Authored-By: Claude Opus 4.8 (1M context) <noreply@anthropic.com>

File: ur_gripper_gz/urdf/inc/robotiq_hande_gripper.xacro (robot description, xacro)
@@ -90,8 +90,7 @@
       <limit effort="130" lower="0.002" upper="0.02" velocity="0.15"/>
     </joint>
-    <!-- NOTE (gz): the real Hand-E has one actuator + a mimic finger, but gz Harmonic's
-         physics engine does not support mimic constraints and gz_ros2_control's software
-         mimic is not enforced here. So both fingers are actuated independently and
-         commanded to the same position by the gripper client (see grippers.py). -->
+    <!-- Single-actuator Hand-E: the right finger mimics the actuated finger_joint. This is
+         enforced by gz only with the bullet-featherstone physics engine (the default DART
+         engine has no mimic-constraint support) — the launch selects it. -->
     <joint name="${prefix}hande_right_finger_joint" type="prismatic">
       <origin rpy="0 0 0" xyz="0 0 0.099"/>
@@ -100,4 +99,5 @@
       <axis xyz="1 0 0"/>
       <limit effort="130" lower="0.002" upper="0.02" velocity="0.15"/>
+      <mimic joint="${prefix}finger_joint" multiplier="1" offset="0"/>
     </joint>
   </xacro:macro>

File: ur_gripper_gz/urdf/inc/ur_gripper_hande.ros2_control.xacro (robot description, xacro)
@@ -2,8 +2,8 @@
 <!--
   ros2_control for UR arm + Robotiq Hand-E in gz-sim.
-  Extends ur_description's arm joint block with BOTH Hand-E finger joints, each with a
-  position command interface. gz Harmonic has no mimic-constraint support and
-  gz_ros2_control's software mimic is not enforced here, so the two fingers are driven
-  independently (the client commands both to the same position).
+  Extends ur_description's arm joint block with the single actuated finger_joint.
+  hande_right_finger_joint is a URDF <mimic> of finger_joint, enforced by gz with the
+  bullet-featherstone physics engine (the launch selects it), so it gets state interfaces
+  only — no command interface.
 -->
 <robot xmlns:xacro="http://wiki.ros.org/xacro">
@@ -31,6 +31,7 @@
         </state_interface>
       </joint>
+      <!-- mimic of finger_joint (see robotiq_hande_gripper.xacro), enforced by gz
+           (bullet-featherstone). Mimic joints get state interfaces only, no command. -->
       <joint name="${tf_prefix}hande_right_finger_joint">
-        <command_interface name="position"/>
         <state_interface name="position">
           <param name="initial_value">${finger_initial_position}</param>
