Commit message: ur_gripper_gz: FT sensor + Cartesian compliance in gz (Spike 2)
Add a wrist force-torque sensor and the FZI cartesian_compliance_controller
to the Hand-E gz bringup, wire FT filtering/zeroing, and fix a hang in the
compliance example.

- FT sensor: gz force_torque sensor (tcp_fts_sensor) on wrist_3_joint plus the
  gz-sim-forcetorque-system plugin (stock empty.sdf omits it), read by
  force_torque_sensor_broadcaster and published on /wrench (remapped from
  ~/wrench). Matching <sensor> block added to the ros2_control xacro.
- Cartesian compliance: cartesian_compliance_controller loaded inactive,
  switched on by ur_control's CompliantController; its ft_sensor_wrench reads
  the gravity-compensated /wrench/filtered.
- ft_filter: bringup runs ur_control_examples/ft_filter, publishing
  /wrench/filtered + a zero_ftsensor service that tares the distal-mass bias.
- Fix compliance-example hang: Arm.zero_ft_sensor() called a UR-driver-only
  service that never exists in sim, and the no-timeout client.call() blocked
  forever. __init_ft_sensor__ now binds FT service lambdas only when
  wait_for_service succeeds; the example declares use_gazebo_sim/use_real_robot.
- COLCON_IGNORE the ROS 1 / MoveIt 1 packages so the workspace builds.

Verified in gz (headless): /wrench at 500 Hz; compliance controller tracks
pose + force, stops on target force, and switches back to the JTC cleanly.

Co-Authored-By: Claude Opus 4.8 <noreply@anthropic.com>

File: ur_gripper_gz/urdf/inc/ur_gripper_hande.ros2_control.xacro (robot description, xacro)
@@ -22,4 +22,17 @@
         tf_prefix="${tf_prefix}"
         initial_positions="${initial_positions}"/>
+      <!-- Wrist force-torque sensor. Mirrors the real ur_robot_driver tcp_fts_sensor
+           (force.x..torque.z). gz_ros2_control's GazeboSimSystem backs these state
+           interfaces from the gz force_torque sensor of the SAME name (tcp_fts_sensor),
+           defined on wrist_3_joint in ur_gripper_hande_gz.urdf.xacro. The
+           force_torque_sensor_broadcaster reads it and publishes /wrench. -->
+      <sensor name="${tf_prefix}tcp_fts_sensor">
+        <state_interface name="force.x"/>
+        <state_interface name="force.y"/>
+        <state_interface name="force.z"/>
+        <state_interface name="torque.x"/>
+        <state_interface name="torque.y"/>
+        <state_interface name="torque.z"/>
+      </sensor>
       <joint name="${tf_prefix}finger_joint">
         <command_interface name="position"/>

File: ur_gripper_gz/urdf/ur_gripper_2f85_gz.urdf.xacro (robot description, xacro)
@@ -27,5 +27,5 @@
     visual_parameters_file="$(find ur_description)/config/$(arg ur_type)/visual_parameters.yaml"
     safety_limits="false" safety_pos_margin="0.15" safety_k_position="20" force_abs_paths="true">
-    <origin xyz="0 0 0" rpy="0 0 0"/>
+    <origin xyz="0 0 0" rpy="0 0 1.5707"/>
   </xacro:ur_robot>
   <!-- mount the gripper on the UR tool flange -->

File: ur_gripper_gz/urdf/ur_gripper_hande_gz.urdf.xacro (robot description, xacro)
@@ -30,5 +30,5 @@
   <xacro:arg name="spawn_y" default="0.0"/>
   <xacro:arg name="spawn_z" default="0.0"/>
-  <xacro:arg name="spawn_yaw" default="-1.5707"/>
+  <xacro:arg name="spawn_yaw" default="1.5707"/>
   <link name="world"/>
   <xacro:ur_robot
@@ -54,4 +54,24 @@
       </ros>
     </plugin>
+    <!-- gz force_torque sensors are inert without this system (stock empty.sdf does
+         not load it). It scans the world for force_torque sensors, computes each
+         joint's reaction wrench, and publishes it on the sensor's gz topic, which
+         gz_ros2_control auto-discovers and exposes as the tcp_fts_sensor interfaces. -->
+    <plugin filename="gz-sim-forcetorque-system" name="gz::sim::systems::ForceTorque"/>
+  </gazebo>
+  <!-- Wrist force-torque sensor. Attached to wrist_3_joint (a real revolute joint, so
+       bullet-featherstone always models it as a constraint and reports its reaction
+       wrench — a fixed joint at ft_frame would be lumped away). Reported in the child
+       (wrist_3_link) frame; the broadcaster stamps frame_id=wrist_3_link and downstream
+       consumers transform via TF. Name MUST match the <sensor> in the ros2_control xacro. -->
+  <gazebo reference="$(arg tf_prefix)wrist_3_joint">
+    <sensor name="$(arg tf_prefix)tcp_fts_sensor" type="force_torque">
+      <always_on>true</always_on>
+      <update_rate>500</update_rate>
+      <force_torque>
+        <frame>child</frame>
+        <measure_direction>child_to_parent</measure_direction>
+      </force_torque>
+    </sensor>
   </gazebo>
   <!-- Home pose from ur_gripper_hande_cubes.launch spawn joint values -->
