Commit message: Add ur_gripper_gz_moveit_config: MoveIt 2 arm + gripper for gz
New custom, self-contained MoveIt 2 config for the gz robots, parameterized by
ur_type + gripper (one package for Hand-E and 2F-85). Adds the gripper as a
MoveIt planning group / end-effector so MoveIt can actuate it, and consolidates
all MoveIt assets here (moved out of ur_gripper_gz, which is now a pure bringup).

- config/: vendored kinematics / joint_limits / ompl_planning / moveit.rviz
  (from apt ur_moveit_config, now customizable) + per-gripper moveit_controllers:
  Hand-E gripper_controller is a JTC -> FollowJointTrajectory; 2F-85 is a
  GripperActionController -> GripperCommand (gripper_cmd).
- srdf/ur_gripper_gz.srdf.xacro: wraps the UR arm SRDF; per gripper adds the
  disable_collisions plus (when load_gripper) a `gripper` group (actuated joint
  only; mimics follow), open/close states, and an end_effector on tool0.
- launch/ur_moveit.launch.py: move_group + RViz; args ur_type, gripper,
  load_gripper (false = arm-only), launch_rviz. Reads /robot_description from the
  running gz bringup; executes on scaled_joint_trajectory_controller + gripper.

gz-specific fixes baked into the config:
- gripper disable_collisions are mandatory (else start-state self-collision, -10);
- gripper joints need acceleration limits in joint_limits.yaml (else TOTG fails);
- 2F-85 knuckle position lower bound widened to -0.02 (gz rests it at ~-7e-13,
  and Jazzy CheckStartStateBounds hard-fails an out-of-bounds revolute start).

Verified in gz (headless): 2F-85 arm plan+execute AND gripper open<->close via a
MoveGroup goal (error_code=1). Hand-E arm + gripper close work; full finger reopen
is limited by the known gz Hand-E finger model, not the MoveIt config.

Co-Authored-By: Claude Opus 4.8 <noreply@anthropic.com>

File: ur_gripper_gz_moveit_config/srdf/ur_gripper_gz.srdf.xacro (robot description, xacro)
@@ -1,20 +1,36 @@
 <?xml version="1.0" encoding="UTF-8"?>
 <!--
-  MoveIt 2 semantic description for the ur_gripper_gz bringups.
-  Wraps the upstream ur_moveit_config arm SRDF (the `ur_manipulator` planning group +
-  UR self-collision rules) and adds disable_collisions for the gripper links. move_group
-  reads robot_description (arm + gripper) from the running gz bringup's topic, so without
-  these the rigidly-attached gripper links register as start-state self-collisions and every
-  plan is rejected (error -10). This is an ARM-ONLY MoveIt config: the gripper is not a
-  planning group; its links are simply exempted from collision (they never move during arm
-  planning). Pick the set with the `gripper` arg (hande | robotiq_2f85).
+  MoveIt 2 semantic description for the ur_gripper_gz bringups (UR + Robotiq Hand-E / 2F-85).
+  Wraps the upstream ur_moveit_config arm SRDF (the `ur_manipulator` planning group + UR
+  self-collision rules) and adds, per gripper:
+    * disable_collisions for the gripper links — move_group reads robot_description (arm +
+      gripper) from the running gz bringup's topic, so without these the rigidly-attached
+      gripper links register as start-state self-collisions and every plan is rejected (-10);
+    * (when load_gripper) a `gripper` planning group (the single actuated joint; mimics follow
+      via the URDF), open/close group_states, and an end_effector on tool0 — so MoveIt can
+      actuate the gripper.
+  Args:  name (ur_type), gripper (hande | robotiq_2f85), load_gripper (true | false)
 -->
 <robot xmlns:xacro="http://wiki.ros.org/xacro" name="$(arg name)">
   <xacro:arg name="name" default="ur"/>
   <xacro:arg name="gripper" default="hande"/>
+  <xacro:arg name="load_gripper" default="true"/>
   <xacro:include filename="$(find ur_moveit_config)/srdf/ur_macro.srdf.xacro"/>
   <xacro:ur_srdf/>
-  <!-- Robotiq Hand-E -->
+  <!-- ================= Robotiq Hand-E ================= -->
   <xacro:if value="${'$(arg gripper)' == 'hande'}">
+    <xacro:if value="${'$(arg load_gripper)' == 'true'}">
+      <group name="gripper">
+        <joint name="finger_joint"/>
+      </group>
+      <!-- finger_joint (prismatic): 0.002 = open, 0.02 = closed (URDF limits) -->
+      <group_state name="open" group="gripper">
+        <joint name="finger_joint" value="0.002"/>
+      </group_state>
+      <group_state name="close" group="gripper">
+        <joint name="finger_joint" value="0.02"/>
+      </group_state>
+      <end_effector name="hande" parent_link="tool0" group="gripper" parent_group="ur_manipulator"/>
+    </xacro:if>
     <disable_collisions link1="flange" link2="hand_e_link" reason="Adjacent"/>
     <disable_collisions link1="flange" link2="hande_left_finger" reason="Adjacent"/>
@@ -36,6 +52,19 @@
     <disable_collisions link1="robotiq_coupler" link2="wrist_3_link" reason="Adjacent"/>
   </xacro:if>
-  <!-- Robotiq 2F-85 (PickNik robotiq_description + ur_to_robotiq adapter) -->
+  <!-- ================= Robotiq 2F-85 (PickNik robotiq_description + ur_to_robotiq adapter) ================= -->
   <xacro:if value="${'$(arg gripper)' == 'robotiq_2f85'}">
+    <xacro:if value="${'$(arg load_gripper)' == 'true'}">
+      <group name="gripper">
+        <joint name="robotiq_85_left_knuckle_joint"/>
+      </group>
+      <!-- knuckle (revolute): 0.0 = open, 0.8 = closed (URDF limits) -->
+      <group_state name="open" group="gripper">
+        <joint name="robotiq_85_left_knuckle_joint" value="0.0"/>
+      </group_state>
+      <group_state name="close" group="gripper">
+        <joint name="robotiq_85_left_knuckle_joint" value="0.8"/>
+      </group_state>
+      <end_effector name="robotiq_2f85" parent_link="tool0" group="gripper" parent_group="ur_manipulator"/>
+    </xacro:if>
     <disable_collisions link1="flange" link2="gripper_mount_link" reason="Adjacent"/>
     <disable_collisions link1="flange" link2="robotiq_85_base_link" reason="Adjacent"/>
