Commit message: ur_gripper_gz: Enable Cartesian compliance for Robotiq 2F-85 gripper
Wire up the `cartesian_compliance_controller` for the 2F-85 gripper in Gazebo,
achieving parity with the Hand-E setup.

This includes:
- Configuring `cartesian_compliance_controller` and `forward_velocity_controller`
  in `ur_gz_2f85_controllers.yaml` with parameters for the 2F-85.
- Adding spawners for these controllers (inactive at startup) in
  `ur_2f85_gz_control.launch.py`, with the compliance controller's FT input
  remapped to `/wrench/filtered`.
- Introducing a `gripper_tip_link` in `ur_gripper_2f85_gz.urdf.xacro` to define
  the end-effector TCP for the compliance controller.

`MIGRATION.md` is updated to reflect the completed 2F-85 compliance and to
clarify the removal of older MoveIt 1 / catkin gripper packages, which are
superseded by the new MoveIt 2 configuration.

File: ur_gripper_gz/urdf/ur_gripper_2f85_gz.urdf.xacro (robot description, xacro)
@@ -35,4 +35,13 @@
     <origin xyz="0 0 0" rpy="0 0 0"/>
   </xacro:robotiq_gripper>
+  <!-- TCP frame for compliance / ur_control clients (ee_link='gripper_tip_link').
+       Offset from tool0 through the ur_to_robotiq adapter + 2F-85 body to the open
+       fingertip center (~172 mm along tool Z). -->
+  <link name="$(arg tf_prefix)gripper_tip_link"/>
+  <joint name="$(arg tf_prefix)gripper_tip_joint" type="fixed">
+    <origin xyz="0 0 0.172" rpy="0 0 0"/>
+    <parent link="$(arg tf_prefix)tool0"/>
+    <child link="$(arg tf_prefix)gripper_tip_link"/>
+  </joint>
   <!-- single gz_ros2_control system: arm joints + the actuated gripper knuckle.
        The 5 gripper mimic joints are enforced by gz (bullet-featherstone) from their
